Commit message: :hammer: Update: move mobile base with action graph

File: src/orion_moveit_config/config/orion.ros2_control.xacro (robot description, xacro)
@@ -9,6 +9,4 @@
                 <param name="joint_commands_topic">/isaac_joint_commands</param>
                 <param name="joint_states_topic">/isaac_joint_states</param>
-                <param name="joint_commands_topic">/isaac_wheel_commands</param>
-                <param name="joint_states_topic">/isaac_wheel_states</param>
             </hardware>
             <joint name="joint_flipper_arm_back_left">
@@ -40,4 +38,25 @@
                 <state_interface name="velocity"/>
             </joint>
+            <!--Wheel 관련 추가함-->
+            <!-- <joint name="joint_wheel_back_left">
+              <command_interface name="velocity"/>
+              <state_interface name="position"/>
+              <state_interface name="velocity"/>
+          </joint>
+          <joint name="joint_wheel_back_right">
+              <command_interface name="velocity"/>
+              <state_interface name="position"/>
+              <state_interface name="velocity"/>
+          </joint>
+          <joint name="joint_wheel_front_left">
+              <command_interface name="velocity"/>
+              <state_interface name="position"/>
+              <state_interface name="velocity"/>
+          </joint>
+          <joint name="joint_wheel_front_right">
+              <command_interface name="velocity"/>
+              <state_interface name="position"/>
+              <state_interface name="velocity"/>
+          </joint> -->
         </ros2_control>
     </xacro:macro>
